Commit message: different sh models added v1.0 v2.0 and v2.0_simple

File: softhands_description/urdf/softhands.xacro (robot description, xacro)
@@ -1,34 +1,72 @@
 <?xml version="1.0"?>
 <robot name="softhands" xmlns:xacro="http://www.ros.org/wiki/xacro">
-	<xacro:include filename="$(find softhands_description)/urdf/v1.0/sh_v1.xacro"/>
-	<xacro:macro name="softhands" params="type version parent model position orientation">
-		# Softhand Base
-		<joint name="${type}_hand_base_joint" type="fixed">
-			<origin xyz="${position}" rpy="${orientation}"/>
-			<parent link="${parent}" />
-			<child link="${type}_hand_palm_base" />
-		</joint>
-		<link name="${type}_hand_palm_base">
-		</link>
-		# Softhand VERSION 1.0
-        <xacro:if value="${version == 'v1.0'}">
-			<xacro:sh_v1 type="${type}"
-				parent = "${parent}"
-				position ="${position}"
-				orientation ="${orientation}">
-			</xacro:sh_v1>
-		</xacro:if>
-		# TODO: OTHER VERSIONs
-		# Gazebo custom synergy-plugin
-	    <gazebo>
-	        <plugin name="synergy_plugin" filename="libsofthands_synergy_plugin.so">
-				<namespace>${type}_hand</namespace>
-				<close_rate>0.001</close_rate> 			# from 0 to 1: 0 - slow closure, 1 - fast closure
-				<close_type>${model}</close_type> 		# hand closure type, "power" or "pinch"
-	        </plugin>
-	    </gazebo>
-		<gazebo>
-		  <self_collide>1</self_collide>
-		</gazebo>
-	</xacro:macro>
+  <xacro:include filename="$(find softhands_description)/urdf/v1.0/sh_v1.xacro"/>
+  <xacro:include filename="$(find softhands_description)/urdf/v2.0/sh_v2.xacro"/>
+  <xacro:include filename="$(find softhands_description)/urdf/v2.0_simple/sh_v2_simple.xacro"/>
+  <material name="qbmove/default">
+    <color rgba="0.35 0.35 0.35 1.0"/>
+  </material>
+  <xacro:macro name="softhands" params="type version parent model position orientation">
+    # Softhand Base
+    <joint name="${type}_hand_base_joint" type="fixed">
+	    <origin xyz="${position}" rpy="${orientation}"/>
+	    <parent link="${parent}" />
+	    <child link="${type}_hand_palm_base" />
+    </joint>
+    <link name="${type}_hand_palm_base">
+    </link>
+    # Softhand VERSION 1.0
+    <xacro:if value="${version == 'v1.0'}">
+	<xacro:sh_v1 type="${type}"
+	    parent = "${parent}"
+	    position ="${position}"
+	    orientation ="${orientation}">
+	</xacro:sh_v1>
+    </xacro:if>
+    # Softhand VERSION 2.0
+    <xacro:if value="${version == 'v2.0'}">
+      <xacro:sh_v2 type="${type}"
+	      parent = "${parent}"
+	      position ="${position}"
+	      orientation ="${orientation}">
+      </xacro:sh_v2>
+    </xacro:if>
+    # Softhand VERSION 2.0 SIMPLIFIED (less joints)
+    <xacro:if value="${version == 'v2.0_simple'}">
+      <xacro:sh_v2_simple type="${type}"
+	      parent = "${parent}"
+	      position ="${position}"
+	      orientation ="${orientation}">
+      </xacro:sh_v2_simple>
+    </xacro:if>
+    # TODO: OTHER VERSIONs
+<!--     # Gazebo custom synergy-plugin
+    <gazebo>
+	<plugin name="synergy_plugin" filename="libsofthands_synergy_plugin.so">
+			<namespace>${type}_hand</namespace>
+			<close_rate>0.001</close_rate> 			# from 0 to 1: 0 - slow closure, 1 - fast closure
+			<close_type>${model}</close_type> 		# hand closure type, "power" or "pinch"
+	</plugin>
+    </gazebo> -->
+    # Gazebo NEW custom synergy-plugin
+<!--     <gazebo>
+            <plugin name="synergy_plugin" filename="libsofthand_mimic_plugin.so">
+                        <namespace>right_hand</namespace>
+                        <operation_mode>0</operation_mode>
+                        <spring_k>10</spring_k>
+                        <spring_k_mimic>0.5</spring_k_mimic>
+            </plugin>
+    </gazebo> -->
+    <gazebo>
+            <plugin name="synergy_plugin" filename="libsofthand_plugin.so">
+                        <namespace>right_hand</namespace>
+                        <operation_mode>2</operation_mode>
+                        <spring_k>20</spring_k>
+                        <spring_k_tendon>100</spring_k_tendon>
+            </plugin>
+    </gazebo>
+    <gazebo>
+      <self_collide>1</self_collide>
+    </gazebo>
+  </xacro:macro>
 </robot>

File: softhands_description/urdf/test_SHs.urdf.xacro (robot description, xacro)
@@ -2,11 +2,22 @@
 <robot name="test_SHs" xmlns:xacro="http://www.ros.org/wiki/xacro">
 	<xacro:include filename="$(find softhands_description)/urdf/softhands.xacro"/>
- 	<gazebo reference="root_link">
-		<material>Gazebo/Orange</material>
-	</gazebo>
-	<link name="root_link"/>
-<!-- 	<joint name="object_joint" type="floating">
-		<origin xyz="0.14 0.03 -0.05" rpy="0 0 0"/>
-		<parent link="root_link" />
+	<!--<xacro:softhands type="right"
+	  version = "v1.0"
+	  parent = "root_link"
+	  position ="0 0 0"
+	  orientation ="0 1.57 0"
+	  model = "power">
+	</xacro:softhands>-->
+<!--	<xacro:softhands type="left"
+	  version = "v1.0"
+	  parent = "root_link"
+	  position="0 0.4 0"
+	  orientation="0 1.57 0"
+	  model = "pinch">
+	</xacro:softhands>-->
+	<link name="world"/>
+<!--     <joint name="object_joint" type="fixed">
+		<origin xyz="0.04 0.03 0.11" rpy="0 0 0"/>
+		<parent link="world" />
 		<child link="object" />
 	</joint>
@@ -29,18 +40,25 @@
 			</geometry>
 		</collision>
-	</link>  -->
+	</link>  --> -->
+<!-- 	<xacro:softhands type="right"
+		version = "v1.0"
+ 		parent = "world"
+		position ="0 0 0"
+		orientation ="0 0.0 0"
+		model = "power">
+	</xacro:softhands> -->
 	<xacro:softhands type="right"
-		version = "v1.0"
- 		parent = "root_link"
+		version = "v2.0_simple"
+ 		parent = "world"
 		position ="0 0 0"
-		orientation ="0 1.57 0"
+		orientation ="0 0.0 0"
 		model = "power">
 	</xacro:softhands>
-	<xacro:softhands type="left"
-		version = "v1.0"
- 		parent = "root_link"
-		position="0 0.4 0"
-		orientation="0 1.57 0"
-		model = "pinch">
-	</xacro:softhands>
+<!-- 	<xacro:softhands type="right"
+		version = "v2.0"
+ 		parent = "world"
+		position ="0 0 0"
+		orientation ="0 0 0"
+		model = "power">
+	</xacro:softhands> -->
 </robot>

File: softhands_description/urdf/v1.0/finger.xacro (robot description, xacro)
@@ -1,5 +1,5 @@
 <?xml version="1.0"?>
 <robot xmlns:xacro="http://www.ros.org/wiki/xacro">
-  <xacro:macro name="finger" params="type ns sign position orientation">
+  <xacro:macro name="finger_v1" params="type ns sign position orientation">
     <!-- KNUCKLE -->
     <joint name="${ns}_${type}_abd_joint" type="revolute">

File: softhands_description/urdf/v1.0/sh_v1.xacro (robot description, xacro)
@@ -42,38 +42,38 @@
 			</link>
 			# Thumb finger
-			<xacro:thumb type="thumb"
+			<xacro:thumb_v1 type="thumb"
 		 		ns = "${type}_hand"
 		 		sign = "1"
 				position="0.00566972 0.0296160 0.0553140"
 				orientation="0.0 -0.38397275793662144 1.5707963267948966">
-			</xacro:thumb>
+			</xacro:thumb_v1>
 			# Index finger
-			<xacro:finger type="index"
+			<xacro:finger_v1 type="index"
 				ns = "${type}_hand"
 				sign = "1"
 				position="-0.0033 0.0195 0.0936994"
 				orientation="1.5707963267948966 -1.4835299330931884 1.5707963267948966">
-			</xacro:finger>
+			</xacro:finger_v1>
 			# Middle finger
-			<xacro:finger type="middle"
+			<xacro:finger_v1 type="middle"
 				ns = "${type}_hand"
 				sign = "1"
 				position="-0.003300000 0.0 0.100699"
 				orientation="3.141592 -1.5707963267948966 0.0">
-			</xacro:finger>
+			</xacro:finger_v1>
 		 	# Ring finger
-		 	<xacro:finger type="ring"
+		 	<xacro:finger_v1 type="ring"
 		 		ns = "${type}_hand"
 		 		sign = "1"
 				position="-0.0033 -0.0195 0.0936994"
 				orientation="-1.5707963267948966 -1.5184364298870514 -1.5707963267948966">
-			</xacro:finger>
+			</xacro:finger_v1>
 		 	# Little finger
-		 	<xacro:finger type="little"
+		 	<xacro:finger_v1 type="little"
 		 		ns = "${type}_hand"
 		 		sign = "1"
 				position="-0.0033 -0.039 0.0836994"
 				orientation="-1.5707963267948966 -1.4835299330931884 -1.5707963267948966">
-			</xacro:finger>
+			</xacro:finger_v1>
 		</xacro:if>
 		# LEFT HAND

File: softhands_description/urdf/v1.0/thumb.xacro (robot description, xacro)
@@ -1,5 +1,5 @@
 <?xml version="1.0"?>
 <robot xmlns:xacro="http://www.ros.org/wiki/xacro">
-  <xacro:macro name="thumb" params="type ns sign position orientation">
+  <xacro:macro name="thumb_v1" params="type ns sign position orientation">
     <!-- KNUCKLE -->
     <joint name="${ns}_${type}_abd_joint" type="continuous">
